File: dvideoboard/dvideoboard.sch (KiCad schematic (older format))
At the start: 18 parts, among them IC1 LVC245A, IC2 LVC245A, IC3 LVC245A, IC4 LVC245A, P1 CONN_02X16, P3 JTAG, U1 10M08SC, U2 ADV7513, U3 TC1262-33VDB, U4 TC1262-33VDB, U5 Si501

Commit message: Ongoing development fpga board
Parts:
- removed U3, U4: TC1262-33VDB, TO_SOT_Packages_SMD:SOT-223, symbol TC1262-33VDB
- removed U5: Si501, Oscillators:Oscillator_SMD_SeikoEpson_SG8002LB-4pin_5.0x3.2mm_HandSoldering, symbol Si501
- added C10: 4.7uF, Capacitors_SMD:C_0805, symbol C_Small
- added C11, C12, C6, C9: 10uF, Capacitors_SMD:C_0805, symbol C_Small
- added C7: 47u, Capacitors_SMD:C_1206, symbol C_Small
- added C8: 4.7u, Capacitors_SMD:C_0805, symbol C_Small
- added D2: LED, LEDs:LED_0805, symbol Led_Small
- added F1: 0ZCK0050AF2E, Capacitors_SMD:C_0805, symbol F_Small
- added IC5, IC6: EP5388QI, Housings_SSOP:TSSOP-16_4.4x5mm_Pitch0.65mm, symbol EP5388QI
- added L1, L2, L3, L4, L5, L6, L7: 10uH, Capacitors_SMD:C_0805, symbol INDUCTOR_SMALL
- added P2: POWER, Pin_Headers:Pin_Header_Straight_1x02_Pitch2.54mm, symbol CONN_02X01
- added P4: HDMI-A, footprints:FCI_10029449-11-5B13-5DRLF, symbol HDMI-A
- added P5: CONN_01X02, Pin_Headers:Pin_Header_Straight_2x01_Pitch2.54mm, symbol CONN_01X02
- added R10, R11, R13, R14, R15: 2K, Resistors_SMD:R_0805, symbol R_Small
- added R12, R2, R3, R4, R5, R6, R7, R8: 10k, Resistors_SMD:R_0805, symbol R_Small
- added R16: 1K, Resistors_SMD:R_0805, symbol R_Small
- added R9: 887, Resistors_SMD:R_0805, symbol R_Small
- added U3: TG2016SBN 20.0000M-TCGNNM3, Crystals:Crystal_SMD_2016-4pin_2.0x1.6mm, symbol TG2016SBN
- C1, C2, C3, C4, C5: value 100n -> 10uF; footprint Capacitors_SMD:C_0805_HandSoldering -> Capacitors_SMD:C_0805
- D1: value Led_Small -> LED
- IC1, IC2, IC3, IC4: value LVC245A -> SN74LVC245APWR
- R1: footprint Resistors_SMD:R_0805_HandSoldering -> Resistors_SMD:R_0805
- U1: value 10M08SC -> 10M08SCE144C8G; footprint eqfp144:QFP_144_GND -> footprints:QFP_144_GND
Connections:
- net labels added: +5V, 1V8A, 1V8B, 1V8C, 3V3A, 3V3B, 3V3C, 3V3D
- wire segments 340 -> 535
- no-connect marks 4 -> 31
Other:
- moved on the sheet: D1, P3, R1

Commit message: finished pcb design
Parts:
- removed IC5, IC6: EP5388QI, Housings_SSOP:TSSOP-16_4.4x5mm_Pitch0.65mm, symbol EP5388QI
- removed P5: CONN_01X02, Pin_Headers:Pin_Header_Straight_2x01_Pitch2.54mm, symbol CONN_01X02
- added C13, C14, C15, C16, C17, C18, C19, C20, C21, C22, C23, C24, C25, C26, C27, C28, C29, C30, C31, C32, C33, C34, C35, C36, C37, C38, C39, C40, C41, C42, C43: 100nF, Capacitors_SMD:C_0805_HandSoldering, symbol C_Small
- added IC5, IC6: AP3417C, TO_SOT_Packages_SMD:TSOT-23-5_HandSoldering, symbol AP3417C
- added L8, L9: 2.2uH, Capacitors_SMD:C_0805_HandSoldering, symbol INDUCTOR_SMALL
- added P5: CONN_01X03, Pin_Headers:Pin_Header_Straight_1x03_Pitch2.54mm, symbol CONN_01X03
- added R17: 450k, Resistors_SMD:R_0805_HandSoldering, symbol R_Small
- added R18, R20: 100k, Resistors_SMD:R_0805_HandSoldering, symbol R_Small
- added R19: 200k, Resistors_SMD:R_0805_HandSoldering, symbol R_Small
- C1, C11, C12, C2, C3, C4, C5, C6, C8, C9, F1, L1, L2, L3, L4, L5, L6, L7: footprint Capacitors_SMD:C_0805 -> Capacitors_SMD:C_0805_HandSoldering
- C10: value 4.7uF -> 4.7u; footprint Capacitors_SMD:C_0805 -> Capacitors_SMD:C_0805_HandSoldering
- C7: footprint Capacitors_SMD:C_1206 -> Capacitors_SMD:C_1206_HandSoldering
- R1, R10, R11, R12, R13, R14, R15, R16, R2, R3, R4, R5, R6, R7, R8, R9: footprint Resistors_SMD:R_0805 -> Resistors_SMD:R_0805_HandSoldering
Connections:
- wire segments 535 -> 614
- no-connect marks 31 -> 29
Other:
- moved on the sheet: C8

Commit message: first working program on the dvideo-board (lead blinker)
Parts:
- removed U3: TG2016SBN 20.0000M-TCGNNM3, Crystals:Crystal_SMD_2016-4pin_2.0x1.6mm, symbol TG2016SBN
- added C44, C45: 100nF, Capacitors_SMD:C_0805_HandSoldering, symbol C_Small
- added R21: 10k, Resistors_SMD:R_0805_HandSoldering, symbol R_Small
- added SW1: SKRWAEE030, Buttons_Switches_SMD:SW_SPST_EVPBF, symbol SW_PUSH_SMALL_H
- added U3: LFSPXO025560, Crystals:Crystal_SMD_EuroQuartz_MT-4pin_3.2x2.5mm_HandSoldering, symbol LFSPXO025560
- R17: value 450k -> 450k 1%
- R18, R20: value 100k -> 100k 1%
- R19: value 200k -> 200k 1%
- R9: value 887 -> 887 1%
Connections:
- wire segments 614 -> 625
- no-connect marks 29 -> 27
Other:
- moved on the sheet: C18, C19, C20, C21, C22, C23, C24, C25, C26, C27, C28, C29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
