File: dvideoboard/rev2/dvideoboard.kicad_pcb (KiCad board)
At the start: 2 copper layers, 61 x 43.2 mm, 82 parts, among them IC1 AP3417C, IC2 AP3417C, P1 CONN_02X16, P2 JTAG, P3 POWER, P4 HDMI-A, U1 10M08SCE144C8G, U2 LFSPXO025560, U3 ADV7513

Commit message: Rev. 2  Gerber files
Parts:
- removed C42: 10uF, Capacitors_SMD:C_0805_HandSoldering
- C27, C38: value 4.7u -> 10uF
Routing:
- net +5V: track 99.0 -> 97.3 mm, vias 4 -> 3
Other:
- board text added: "2017-04-10 github.com/ c0pperdragon"
- board text removed: "2017-04-08 github.com/ c0pperdragon"
Changed lines of the file:
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@@
 (kicad_pcb (version 4) (host pcbnew 4.0.4-stable)
   (general
-    (links 321)
+    (links 319)
     (no_connects 0)
     (area 88.824999 43.104999 149.935001 86.435001)
     (thickness 1.6)
     (drawings 30)
-    (tracks 1184)
+    (tracks 1180)
     (zones 0)
-    (modules 82)
+    (modules 81)
     (nets 133)
   )
   (page A4)
   (layers
-    (0 F.Cu signal hide)
-    (31 B.Cu signal)
+    (0 F.Cu signal)
+    (31 B.Cu signal hide)
     (32 B.Adhes user)
     (33 F.Adhes user)
@@
     (35 F.Paste user)
     (36 B.SilkS user)
-    (37 F.SilkS user hide)
+    (37 F.SilkS user)
     (38 B.Mask user)
     (39 F.Mask user)
@@
   )
   (setup
-    (last_trace_width 0.5)
+    (last_trace_width 0.25)
     (user_trace_width 0.5)
     (user_trace_width 0.75)
@@
     (solder_mask_min_width 0.2)
     (aux_axis_origin 0 0)
-    (visible_elements 7FFEBFFF)
+    (visible_elements 7FFEFFFF)
     (pcbplotparams
       (layerselection 0x010f0_80000001)
@@
       (effects (font (size 1 1) (thickness 0.15)))
     )
-    (fp_text value 4.7u (at 0 1.75) (layer F.Fab)
+    (fp_text value 10uF (at 0 1.75) (layer F.Fab)
       (effects (font (size 1 1) (thickness 0.15)))
     )
@@
       (effects (font (size 1 1) (thickness 0.15)))
     )
-    (fp_text value 4.7u (at 0 1.75) (layer F.Fab)
+    (fp_text value 10uF (at 0 1.75) (layer F.Fab)
       (effects (font (size 1 1) (thickness 0.15)))
     )
@@
   (module footprints:QFP_144_GND (layer F.Cu)
     (at 110.49 55.88 90)
-    (fp_text reference U1 (at 0 -12.9 90) (layer F.SilkS) hide
+    (fp_text reference U1 (at 0 -12.9 90) (layer F.SilkS)
       (effects (font (size 1.2 1.2) (thickness 0.15)))
     )
@@
     )
   )
-  (module Capacitors_SMD:C_0805_HandSoldering (layer B.Cu)
-    (at 128.27 82.55 90)
-    (descr "Capacitor SMD 0805, hand soldering")
-    (tags "capacitor 0805")
-    (attr smd)
-    (fp_text reference C42 (at 0.127 -1.651 90) (layer B.SilkS)
-      (effects (font (size 1 1) (thickness 0.15)) (justify mirror))
-    )
-    (fp_text value 10uF (at 0 -1.75 90) (layer B.Fab)
-      (effects (font (size 1 1) (thickness 0.15)) (justify mirror))
-    )
-    (fp_text user %R (at 0.127 -1.651 90) (layer B.Fab)
-      (effects (font (size 1 1) (thickness 0.15)) (justify mirror))
-    )
-    (fp_line (start -1 -0.62) (end -1 0.62) (layer B.Fab) (width 0.1))
-    (fp_line (start 1 -0.62) (end -1 -0.62) (layer B.Fab) (width 0.1))
-    (fp_line (start 1 0.62) (end 1 -0.62) (layer B.Fab) (width 0.1))
-    (fp_line (start -1 0.62) (end 1 0.62) (layer B.Fab) (width 0.1))
-    (fp_line (start 0.5 0.85) (end -0.5 0.85) (layer B.SilkS) (width 0.12))
-    (fp_line (start -0.5 -0.85) (end 0.5 -0.85) (layer B.SilkS) (width 0.12))
-    (fp_line (start -2.25 0.88) (end 2.25 0.88) (layer B.CrtYd) (width 0.05))
-    (fp_line (start -2.25 0.88) (end -2.25 -0.87) (layer B.CrtYd) (width 0.05))
-    (fp_line (start 2.25 -0.87) (end 2.25 0.88) (layer B.CrtYd) (width 0.05))
-    (fp_line (start 2.25 -0.87) (end -2.25 -0.87) (layer B.CrtYd) (width 0.05))
-    (pad 1 smd rect (at -1.25 0 90) (size 1.5 1.25) (layers B.Cu B.Paste B.Mask)
-      (net 39 +5V))
-    (pad 2 smd rect (at 1.25 0 90) (size 1.5 1.25) (layers B.Cu B.Paste B.Mask)
-      (net 33 GND))
-    (model Capacitors_SMD.3dshapes/C_0805.wrl
-      (at (xyz 0 0 0))
-      (scale (xyz 1 1 1))
-      (rotate (xyz 0 0 0))
-    )
-  )
   (module Capacitors_SMD:C_0603_HandSoldering (layer B.Cu)
     (at 122.174 63.881)
@@
       (xy 0.555814 -2.531069)) (layer F.SilkS) (width 0.01))
   )
-  (gr_text "2017-04-08\ngithub.com/\nc0pperdragon" (at 117.983 81.534) (layer B.SilkS)
+  (gr_text "2017-04-10\ngithub.com/\nc0pperdragon" (at 117.983 81.534) (layer B.SilkS)
     (effects (font (size 1.5 1.5) (thickness 0.3)) (justify mirror))
   )
@@
   (segment (start 134.3 80.45) (end 136.8 80.45) (width 0.25) (layer F.Cu) (net 4))
   (segment (start 125.575 47.378) (end 124.594 47.378) (width 0.25) (layer F.Cu) (net 17))
-  (segment (start 124.594 47.378) (end 122.047 44.831) (width 0.25) (layer F.Cu) (net 17))
-  (via (at 122.047 44.831) (size 0.6) (drill 0.4) (layers F.Cu B.Cu) (net 17))
-  (segment (start 122.047 44.831) (end 112.014 44.831) (width 0.25) (layer B.Cu) (net 17))
-  (segment (start 112.014 44.831) (end 111.76 45.085) (width 0.25) (layer B.Cu) (net 17))
+  (segment (start 124.594 47.378) (end 122.174 44.577) (width 0.25) (layer F.Cu) (net 17))
+  (via (at 122.174 44.577) (size 0.6) (drill 0.4) (layers F.Cu B.Cu) (net 17))
+  (segment (start 122.174 44.577) (end 112.141 44.577) (width 0.25) (layer B.Cu) (net 17))
+  (segment (start 112.141 44.577) (end 111.76 45.085) (width 0.25) (layer B.Cu) (net 17))
   (segment (start 111.76 45.085) (end 111.76 46.228) (width 0.25) (layer B.Cu) (net 17))
   (via (at 111.76 46.228) (size 0.6) (drill 0.4) (layers F.Cu B.Cu) (net 17))
@@
   (segment (start 148.209 46.228) (end 148.209 49.149) (width 0.5) (layer F.Cu) (net 37))
   (segment (start 128.425 45.078) (end 128.425 47.378) (width 0.5) (layer F.Cu) (net 37))
-  (segment (start 135.89 45.64) (end 133.35 45.64) (width 0.5) (layer F.Cu) (net 37) (status 20))
-  (segment (start 133.35 45.64) (end 132.501 44.791) (width 0.5) (layer F.Cu) (net 37) (status 10))
   (segment (start 132.501 44.791) (end 132.48 44.77) (width 0.5) (layer F.Cu) (net 37) (status 10))
   (segment (start 128.733 44.77) (end 128.425 45.078) (width 0.5) (layer F.Cu) (net 37))
+  (segment (start 135.89 45.64) (end 133.35 45.64) (width 0.5) (layer F.Cu) (net 37) (status 20))
+  (segment (start 133.35 45.64) (end 132.501 44.791) (width 0.5) (layer F.Cu) (net 37) (status 10))
   (via (at 127.695 66.421) (size 0.6) (drill 0.4) (layers F.Cu B.Cu) (net 38))
   (segment (start 126.746 66.482) (end 127.634 66.482) (width 0.25) (layer B.Cu) (net 38))
@@
   (segment (start 120.63 82.657) (end 120.97 82.997) (width 0.75) (layer F.Cu) (net 39))
   (segment (start 120.97 82.997) (end 120.63 82.55) (width 0.75) (layer F.Cu) (net 39))
-  (via (at 129.667 84.55) (size 0.6) (drill 0.4) (layers F.Cu B.Cu) (net 39))
-  (segment (start 128.27 83.8) (end 129.052 84.582) (width 1) (layer B.Cu) (net 39))
-  (segment (start 129.635 84.582) (end 129.052 84.582) (width 1) (layer B.Cu) (net 39))
-  (segment (start 129.635 84.582) (end 129.667 84.55) (width 1) (layer B.Cu) (net 39))
   (segment (start 130.81 83.8) (end 131.592 84.582) (width 1) (layer B.Cu) (net 39))
   (segment (start 141.525 49.45) (end 144.907 52.832) (width 0.5) (layer F.Cu) (net 39) (status 10))
@@
   (segment (start 139.78 68.58) (end 140.22 69.02) (width 0.25) (layer F.Cu) (net 54))
   (segment (start 135.195 68.58) (end 139.62 68.58) (width 0.25) (layer F.Cu) (net 54))
-  (segment (start 124.079 48.895) (end 123.314 48.13) (width 0.25) (layer F.Cu) (net 56))
   (segment (start 133.35 51.054) (end 131.191 48.895) (width 0.25) (layer F.Cu) (net 56))
-  (segment (start 131.191 48.895) (end 124.079 48.895) (width 0.25) (layer F.Cu) (net 56))
-  (segment (start 123.314 48.13) (end 121.49 48.13) (width 0.25) (layer F.Cu) (net 56))
   (segment (start 133.35 51.054) (end 133.858 51.054) (width 0.25) (layer F.Cu) (net 56))
-  (segment (start 134.195 51.899) (end 134.195 55.895) (width 0.25) (layer F.Cu) (net 56))
-  (segment (start 134.195 51.391) (end 134.195 51.899) (width 0.25) (layer F.Cu) (net 56))
   (segment (start 133.858 51.054) (end 134.195 51.391) (width 0.25) (layer F.Cu) (net 56))
   (segment (start 133.35 48.34) (end 133.35 51.054) (width 0.25) (layer F.Cu) (net 56) (status 10))
+  (segment (start 124.079 48.895) (end 123.314 48.13) (width 0.25) (layer F.Cu) (net 56))
+  (segment (start 131.191 48.895) (end 124.079 48.895) (width 0.25) (layer F.Cu) (net 56))
+  (segment (start 134.195 51.391) (end 134.195 51.899) (width 0.25) (layer F.Cu) (net 56))
+  (segment (start 123.314 48.13) (end 121.49 48.13) (width 0.25) (layer F.Cu) (net 56))
+  (segment (start 134.195 51.899) (end 134.195 55.895) (width 0.25) (layer F.Cu) (net 56))
   (segment (start 96.139 79.121) (end 96.774 78.486) (width 0.25) (layer F.Cu) (net 57))
   (segment (start 100.457 78.74) (end 112.776 78.74) (width 0.25) (layer F.Cu) (net 57))
