File: dvideoboard/rev2/dvideoboard.sch (KiCad schematic (older format))
At the start: 78 parts, among them IC1 AP3417C, IC2 AP3417C, P1 CONN_02X16, P2 JTAG, P3 POWER, P4 HDMI-A, U1 10M08SCE144C8G, U2 LFSPXO025560, U3 ADV7513

Commit message: Rev. 2  Gerber files
Parts:
- removed C42: 10uF, Capacitors_SMD:C_0805_HandSoldering, symbol C_Small
- C27, C38: value 4.7u -> 10uF
Connections:
- wire segments 535 -> 533

Commit message: Resume work on upscaler
Parts:
- C1, C10, C11, C12, C13, C14, C15, C16, C17, C18, C19, C2, C20, C21, C22, C23, C24, C25, C26, C27, C28, C29, C3, C30, C31, C32, C33, C34, C35, C36, C37, C38, C39, C4, C40, C41, C43, C5, C6, C7, C8, C9: symbol C_Small -> Device:C_Small
- IC1, IC2: symbol AP3417C -> components:AP3417C
- L1, L2, L3, L4, L5, L6, L7, L8, L9: symbol INDUCTOR_SMALL -> dvideoboard-rescue:INDUCTOR_SMALL
- P1: symbol CONN_02X16 -> dvideoboard-rescue:CONN_02X16
- P2: symbol CONN_02X05 -> dvideoboard-rescue:CONN_02X05
- P3: symbol CONN_02X01 -> dvideoboard-rescue:CONN_02X01
- P4: symbol HDMI-A -> components:HDMI-A
- R1, R10, R11, R12, R13, R14, R15, R17, R18, R2, R3, R4, R5, R6, R7, R8, R9: symbol R_Small -> Device:R_Small
- U1: symbol 10M08SC -> components:10M08SC
- U2: symbol LFSPXO025560 -> components:LFSPXO025560
- U3: symbol ADV7513 -> components:ADV7513
Connections:
- wire segments 533 -> 632
